File: CAN Knoten/Schaltplan.sch (EAGLE design)
At the start: 39 parts, among them IC1 74LS165D, IC2 74LS165D, K1 68711614522, K2 68711614522, K3 68711614522, K4 68711614522, Q1 HC49-U - 16MHz, Q2 HC49-U - xMHz

Commit message: 
Parts:
- added R6: 10k, rcl:R-EU_R1206
- added XW1: (no value), Atmel - ISP_6 (AVR ISP MKII):WSL6
Connections:
- new net N$31: D1.PDI_CLOCK(!RESET!), R6.1, XW1.RESET
- new net XMEGA_PDI_DATA: D1.PDI_DATA, XW1.MISO
- net GND: now also XW1.GND
- net VCC: now also R6.2, XW1.VCC
Changed lines of the file:
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@@
 <?xml version="1.0" encoding="utf-8"?>
 <!DOCTYPE eagle SYSTEM "eagle.dtd">
-<eagle version="7.7.0">
+<eagle version="6.5.0">
 <drawing>
 <settings>
@@
 <setting verticaltext="up"/>
 </settings>
-<grid distance="0.1" unitdist="inch" unit="mm" style="lines" multiple="1" display="no" altdistance="0.01" altunitdist="inch" altunit="inch"/>
+<grid distance="0.1" unitdist="inch" unit="inch" style="lines" multiple="1" display="no" altdistance="0.01" altunitdist="inch" altunit="inch"/>
 <layers>
 <layer number="1" name="Top" color="4" fill="1" visible="no" active="no"/>
@@
 <part name="LED5" library="led" deviceset="LED" device="SML1206"/>
 <part name="R5" library="rcl" deviceset="R-EU_" device="R1206" value="560R"/>
+<part name="XW1" library="Atmel - ISP_6   (AVR ISP MKII)" deviceset="WSL" device="6"/>
+<part name="R6" library="rcl" deviceset="R-EU_" device="R1206" value="10k"/>
+<part name="P+8" library="supply1" deviceset="VCC" device=""/>
+<part name="GND14" library="supply1" deviceset="GND" device=""/>
 </parts>
 <sheets>
@@
 <instance part="LED5" gate="G$1" x="-154.94" y="-162.56"/>
 <instance part="R5" gate="G$1" x="-154.94" y="-152.4" rot="R90"/>
+<instance part="XW1" gate="G$$1" x="-165.1" y="137.16"/>
+<instance part="R6" gate="G$1" x="-205.74" y="139.7" rot="R90"/>
+<instance part="P+8" gate="VCC" x="-205.74" y="149.86"/>
+<instance part="GND14" gate="1" x="-149.86" y="127"/>
 </instances>
 <busses>
@@
 <pinref part="P+15" gate="VCC" pin="VCC"/>
 </segment>
+<segment>
+<pinref part="XW1" gate="G$$1" pin="VCC"/>
+<wire x1="-152.4" y1="139.7" x2="-149.86" y2="139.7" width="0.1524" layer="91"/>
+<wire x1="-149.86" y1="139.7" x2="-149.86" y2="147.32" width="0.1524" layer="91"/>
+<pinref part="R6" gate="G$1" pin="2"/>
+<wire x1="-205.74" y1="144.78" x2="-205.74" y2="147.32" width="0.1524" layer="91"/>
+<pinref part="P+8" gate="VCC" pin="VCC"/>
+<wire x1="-149.86" y1="147.32" x2="-205.74" y2="147.32" width="0.1524" layer="91"/>
+<junction x="-205.74" y="147.32"/>
+</segment>
 </net>
 <net name="GND" class="0">
@@
 <pinref part="GND12" gate="1" pin="GND"/>
 <junction x="-129.54" y="-116.84"/>
+</segment>
+<segment>
+<pinref part="XW1" gate="G$$1" pin="GND"/>
+<wire x1="-152.4" y1="134.62" x2="-149.86" y2="134.62" width="0.1524" layer="91"/>
+<wire x1="-149.86" y1="134.62" x2="-149.86" y2="129.54" width="0.1524" layer="91"/>
+<pinref part="GND14" gate="1" pin="GND"/>
 </segment>
 </net>
@@
 </segment>
 </net>
+<net name="N$31" class="0">
+<segment>
+<pinref part="R6" gate="G$1" pin="1"/>
+<pinref part="XW1" gate="G$$1" pin="RESET"/>
+<wire x1="-177.8" y1="134.62" x2="-205.74" y2="134.62" width="0.1524" layer="91"/>
+<pinref part="D1" gate="G$1" pin="PDI_CLOCK(!RESET!)"/>
+<wire x1="-200.66" y1="119.38" x2="-205.74" y2="119.38" width="0.1524" layer="91"/>
+<wire x1="-205.74" y1="119.38" x2="-205.74" y2="134.62" width="0.1524" layer="91"/>
+<junction x="-205.74" y="134.62"/>
+</segment>
+</net>
+<net name="XMEGA_PDI_DATA" class="0">
+<segment>
+<pinref part="D1" gate="G$1" pin="PDI_DATA"/>
+<wire x1="-200.66" y1="114.3" x2="-226.06" y2="114.3" width="0.1524" layer="91"/>
+<label x="-226.06" y="114.3" size="1.27" layer="95" rot="R180" xref="yes"/>
+</segment>
+<segment>
+<pinref part="XW1" gate="G$$1" pin="MISO"/>
+<wire x1="-177.8" y1="139.7" x2="-180.34" y2="139.7" width="0.1524" layer="91"/>
+<label x="-180.34" y="139.7" size="1.27" layer="95" rot="R180" xref="yes"/>
+</segment>
+</net>
